Commit message: spiral URDF orientation fix

File: assets/spiral_ramp.urdf (robot description, URDF)
Before this commit: robot staircase, 1 links, 1 joints
Links:
- removed link link
- added link stairsLink, mass .0; collision mesh filename=assets/spiral_ramp.obj scale=1 1 1; visual mesh filename=assets/spiral_ramp.obj scale=1 1 1
Joints:
- removed joint fixed_joint
