Commit message: reduce step height from 0.5m to 0.25m

File: assets/stairs.urdf (robot description, URDF)
Before this commit: robot stairs, 5 links, 4 joints
Joints:
- joint stepOne_to_stepTwo: origin xyz=-2 0 0.5 rpy=0 0 0 -> xyz=-2 0 0.25 rpy=0 0 0
- joint stepThree_to_stepFour: origin xyz=-2 0 0.5 rpy=0 0 0 -> xyz=-2 0 0.25 rpy=0 0 0
- joint stepTwo_to_stepThree: origin xyz=-2 0 0.5 rpy=0 0 0 -> xyz=-2 0 0.25 rpy=0 0 0

Commit message: more steps, also closer

File: assets/stairs.urdf (robot description, URDF)
Before this commit: robot stairs, 5 links, 4 joints
Links:
- added link stepFive, mass .0; collision mesh filename=assets/smooth_step.obj scale=1 1 1; visual mesh filename=assets/smooth_step.obj scale=1 1 1
- added link stepSeven, mass .0; collision mesh filename=assets/smooth_step.obj scale=1 1 1; visual mesh filename=assets/smooth_step.obj scale=1 1 1
- added link stepSix, mass .0; collision mesh filename=assets/smooth_step.obj scale=1 1 1; visual mesh filename=assets/smooth_step.obj scale=1 1 1
Joints:
- added joint stepFive_to_stepSix: type fixed, parent stepFive, child stepSix, origin xyz=-1 0 0.25 rpy=0 0 0
- added joint stepFour_to_stepFive: type fixed, parent stepFour, child stepFive, origin xyz=-1 0 0.25 rpy=0 0 0
- added joint stepSix_to_stepSeven: type fixed, parent stepSix, child stepSeven, origin xyz=-1 0 0.25 rpy=0 0 0
- joint stepOne_to_stepTwo: origin xyz=-2 0 0.25 rpy=0 0 0 -> xyz=-1 0 0.25 rpy=0 0 0
- joint stepThree_to_stepFour: origin xyz=-2 0 0.25 rpy=0 0 0 -> xyz=-1 0 0.25 rpy=0 0 0
- joint stepTwo_to_stepThree: origin xyz=-2 0 0.25 rpy=0 0 0 -> xyz=-1 0 0.25 rpy=0 0 0
