Commit message: load ramp into the track

File: assets/track.urdf (robot description, URDF)
Before this commit: robot stairs, 2 links, 1 joints
Links:
- added link ramp, mass .0; collision mesh filename=assets/box_ramp.obj scale=1 1 1; visual mesh filename=assets/box_ramp.obj scale=1 1 1
Joints:
- added joint track_to_ramp: type fixed, parent track, child ramp, origin xyz=-0.55 -3.5 0.0 rpy=0 0 0
